File: pcb/idiot-lights-pcb/idiot-lights-pcb.kicad_sch (KiCad schematic)
At the start: 92 parts, among them Q1 BSS138, Q10 BSS138, Q11 BSS138, Q12 BSS138, Q13 BSS138, Q14 BSS138, Q15 BSS138, Q16 BSS138, Q2 BSS138, Q3 BSS138, Q4 BSS138, Q5 BSS138, Q6 BSS138, Q7 BSS138, Q8 BSS138, Q9 BSS138, SW1 Toggle left indicator, SW2 Toggle right indicator, SW3 Toggle hazard warning, SW4 Break control, SW5 Reset, U1 RaspberryPi_Pico

Commit message: Increase LED resistor values - dim LEDs
Set RPI pico property to THT again
Parts:
- R10, R12, R14, R16, R18, R2, R20, R22, R24, R26, R28, R30, R32, R4, R6, R8: value 330 -> 10k
Changed lines of the file:
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@@
       (effects (font (size 1.27 1.27)) (justify left))
     )
-    (property "Value" "330" (at 209.55 94.615 0)
+    (property "Value" "10k" (at 209.55 94.615 0)
       (effects (font (size 1.27 1.27)) (justify left))
     )
@@
       (effects (font (size 1.27 1.27)) (justify left))
     )
-    (property "Value" "330" (at 133.35 94.615 0)
+    (property "Value" "10k" (at 133.35 94.615 0)
       (effects (font (size 1.27 1.27)) (justify left))
     )
@@
       (effects (font (size 1.27 1.27)) (justify left))
     )
-    (property "Value" "330" (at 171.45 94.615 0)
+    (property "Value" "10k" (at 171.45 94.615 0)
       (effects (font (size 1.27 1.27)) (justify left))
     )
@@
       (effects (font (size 1.27 1.27)) (justify left))
     )
-    (property "Value" "330" (at 171.45 45.085 0)
+    (property "Value" "10k" (at 171.45 45.085 0)
       (effects (font (size 1.27 1.27)) (justify left))
     )
@@
       (effects (font (size 1.27 1.27)) (justify left))
     )
-    (property "Value" "330" (at 228.6 94.615 0)
+    (property "Value" "10k" (at 228.6 94.615 0)
       (effects (font (size 1.27 1.27)) (justify left))
     )
@@
       (effects (font (size 1.27 1.27)) (justify left))
     )
-    (property "Value" "330" (at 247.65 45.085 0)
+    (property "Value" "10k" (at 247.65 45.085 0)
       (effects (font (size 1.27 1.27)) (justify left))
     )
@@
       (effects (font (size 1.27 1.27)) (justify left))
     )
-    (property "Value" "330" (at 133.35 45.085 0)
+    (property "Value" "10k" (at 133.35 45.085 0)
       (effects (font (size 1.27 1.27)) (justify left))
     )
@@
       (effects (font (size 1.27 1.27)) (justify left))
     )
-    (property "Value" "330" (at 209.55 45.085 0)
+    (property "Value" "10k" (at 209.55 45.085 0)
       (effects (font (size 1.27 1.27)) (justify left))
     )
@@
       (effects (font (size 1.27 1.27)) (justify left))
     )
-    (property "Value" "330" (at 152.4 94.615 0)
+    (property "Value" "10k" (at 152.4 94.615 0)
       (effects (font (size 1.27 1.27)) (justify left))
     )
@@
       (effects (font (size 1.27 1.27)) (justify left))
     )
-    (property "Value" "330" (at 266.7 94.615 0)
+    (property "Value" "10k" (at 266.7 94.615 0)
       (effects (font (size 1.27 1.27)) (justify left))
     )
@@
       (effects (font (size 1.27 1.27)) (justify left))
     )
-    (property "Value" "330" (at 266.7 45.085 0)
+    (property "Value" "10k" (at 266.7 45.085 0)
       (effects (font (size 1.27 1.27)) (justify left))
     )
@@
       (effects (font (size 1.27 1.27)) (justify left))
     )
-    (property "Value" "330" (at 190.5 45.085 0)
+    (property "Value" "10k" (at 190.5 45.085 0)
       (effects (font (size 1.27 1.27)) (justify left))
     )
@@
       (effects (font (size 1.27 1.27)) (justify left))
     )
-    (property "Value" "330" (at 152.4 45.085 0)
+    (property "Value" "10k" (at 152.4 45.085 0)
       (effects (font (size 1.27 1.27)) (justify left))
     )
@@
       (effects (font (size 1.27 1.27)) (justify left))
     )
-    (property "Value" "330" (at 190.5 94.615 0)
+    (property "Value" "10k" (at 190.5 94.615 0)
       (effects (font (size 1.27 1.27)) (justify left))
     )
@@
       (effects (font (size 1.27 1.27)) (justify left))
     )
-    (property "Value" "330" (at 247.65 94.615 0)
+    (property "Value" "10k" (at 247.65 94.615 0)
       (effects (font (size 1.27 1.27)) (justify left))
     )
@@
       (effects (font (size 1.27 1.27)) (justify left))
     )
-    (property "Value" "330" (at 228.6 45.085 0)
-      (effects (font (size 1.27 1.27)) (justify left))
-    )
+    (property "Value" "10k" (at 228.6 45.085 0)
+      (effects (font (size 1.27 1.27)) (justify left))
+    )
